File: KiCAD/control/plate.kicad_pcb (KiCad board)
At the start: 2 copper layers, 90 x 40 mm, 30 parts, among them J1 PJ-002, J2 AVR-ISP-6, J3 Pin Header, Q1 IRLZ44N, SW1 Up, SW2 Down, SW3 Select, U1 L7805, U2 ATtiny84A-P, U3 SSD1306

Commit message: Change references to screen resolution
Change screen resolution from 128x32 to 128x64.
Turns out screen resolution is *not* 128x32...oops.
Other:
- board text added: "128x64 SSD1306 Display"
- board text removed: "128x32 SSD1306 Display"
Changed lines of the file:
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@@
 		)
 	)
-	(gr_text "128x32 SSD1306 Display"
+	(gr_text "128x64 SSD1306 Display"
 		(at 182.5 62 0)
 		(layer "F.SilkS")
